File: led-output-board.kicad_sch (KiCad schematic)
At the start: 27 parts, among them J1 DB301V-3.5-3P-GN, J2 DB301V-3.5-3P-GN, J3 DB301V-3.5-3P-GN, J4 DB301V-3.5-3P-GN, J5 DB301V-3.5-3P-GN, J6 DB301V-3.5-3P-GN, J7 DB301V-3.5-3P-GN, J8 DB301V-3.5-3P-GN, U1 SN74LVC8T245PWR

Commit message: Schematic iteration
Parts:
- added J10: DBT50G-9.5-2P, EasyEDA:CONN-TH_2P-P9.50_DBT50G-9.5-2P, symbol EasyEDA:DBT50G-9.5-2P
- added J9: Conn_02x08_Odd_Even, Connector_IDC:IDC-Header_2x08_P2.54mm_Vertical, symbol Connector_Generic:Conn_02x08_Odd_Even
Connections:
- net +3.3V: now also J9.13 (Pin_13)
- net +5V: now also J9.15 (Pin_15)
- net +VIN: now also J10.2
- net GND: now also J10.1, J9.1 (Pin_1), J9.11 (Pin_11), J9.3 (Pin_3), J9.5 (Pin_5), J9.7 (Pin_7), J9.9 (Pin_9)
- net S0_OUT: no longer names the net of U1.14 (B8)
- net S0_OUT: now also R8.1; no longer R1.1
- net S1_OUT: no longer names the net of U1.15 (B7)
- net S1_OUT: now also R7.1; no longer R2.1
- net S2_OUT: no longer names the net of R3.1
- net S2_OUT: now also U1.19 (B3); no longer U1.16 (B6)
- net S3_OUT: no longer names the net of U1.17 (B5)
- net S3_OUT: now also R5.1; no longer R4.1
- net S4_OUT: no longer names the net of U1.18 (B4)
- net S4_OUT: now also R4.1; no longer R5.1
- net S5_OUT: no longer names the net of R6.1
- net S5_OUT: now also U1.16 (B6); no longer U1.19 (B3)
- net S6_OUT: no longer names the net of U1.20 (B2)
- net S6_OUT: now also R2.1; no longer R7.1
- net S7_OUT: no longer names the net of U1.21 (B1)
- net S7_OUT: now also R1.1; no longer R8.1
- net STRING0: no longer names the net of U1.10 (A8)
- net STRING0: now also J9.16 (Pin_16)
- net STRING1: no longer names the net of U1.9 (A7)
- net STRING1: now also J9.14 (Pin_14)
- net STRING2: no longer names the net of U1.8 (A6)
- net STRING2: now also J9.12 (Pin_12)
- net STRING3: no longer names the net of U1.7 (A5)
- net STRING3: now also J9.10 (Pin_10)
- net STRING4: no longer names the net of U1.6 (A4)
- net STRING4: now also J9.8 (Pin_8)
- net STRING5: no longer names the net of U1.5 (A3)
- net STRING5: now also J9.6 (Pin_6)
- net STRING6: no longer names the net of U1.4 (A2)
- net STRING6: now also J9.4 (Pin_4)
- net STRING7: no longer names the net of U1.3 (A1)
- net STRING7: now also J9.2 (Pin_2)
Other:
- moved on the sheet: C1, C2, F1, F2, F3, F4, F5, F6, F7, F8, J1, J2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

Commit message: Getting close on schematic
Parts:
- removed C1, C2: 100nF, PixelBlit:C_0402, symbol PixelBlit:0402,100nF
- removed F1, F2, F3, F4, F5, F6, F7, F8: 1812L400/16GR, EasyEDA:F1812, symbol EasyEDA:1812L400_16GR
- removed J1, J2: DB301V-3.5-3P-GN, PixelBlit:CONN-TH_DB301V-3.5-3P-GN, symbol PixelBlit:DB301V-3.5-3P-GN
- added C1, C2: 100nF, Capacitor_THT:C_Disc_D4.3mm_W1.9mm_P5.00mm, symbol Device:C
- added F1, F2, F3, F4, F5, F6, F7, F8: RUEF400, easyeda2kicad:FUSE-TH_L14.0-W3.0-P5.08-D0.6, symbol easyeda2kicad:RUEF400
- added J10, J9: DB301V-3.5-3P-GN, easyeda2kicad:CONN-TH_DB301V-3.5-3P-GN, symbol PixelBlit:DB301V-3.5-3P-GN
- J1: renamed from J10; footprint EasyEDA:CONN-TH_2P-P9.50_DBT50G-9.5-2P -> easyeda2kicad:CONN-TH_2P-P9.50_DBT50G-9.5-2P; LCSC Part C395958 -> (none)
- J3, J4, J5, J6, J7, J8: footprint PixelBlit:CONN-TH_DB301V-3.5-3P-GN -> easyeda2kicad:CONN-TH_DB301V-3.5-3P-GN
- R1, R2, R3, R4, R5, R6, R7, R8: footprint PixelBlit:R_0402 -> Resistor_THT:R_Axial_DIN0204_L3.6mm_D1.6mm_P2.54mm_Vertical; LCSC C25118 -> (none); Price 0.004USD -> (none); Stock 468126 -> (none)
- U1: footprint PixelBlit:TSSOP-24_L7.8-W4.4-P0.65-LS6.4-BL -> easyeda2kicad:TSSOP-24_L7.8-W4.4-P0.65-LS6.4-BL
- renumbered J9 to J2
Connections:
- net +3.3V: now also C1.1
- net +5V: now also C2.1
- net +VIN: now also F1.1, F2.1, F3.1, F4.1, F5.1, F6.1, F7.1, F8.1
- net GND: now also C1.2, C2.2, J10.3, J9.3
- net at J6.1: now also F4.2
- net at R1.2: now also J3.2
- net at J8.1: now also F6.2
- net at R3.2: now also J5.2; no longer J3.2
- net at J5.1: now also F3.2
- net at J7.1: now also F5.2
- net at R7.2: now also J9.2; no longer J7.2
- net at R4.2: now also J6.2; no longer J4.2
- net at R2.2: now also J4.2
- net at R5.2: now also J7.2; no longer J5.2
- net at R6.2: now also J8.2; no longer J6.2
- net at J3.1: now also F1.2
- net at R8.2: now also J10.2; no longer J8.2
- net at J4.1: now also F2.2
- new net: F7.2, J9.1
- new net: F8.2, J10.1
Other:
- note added: "Capacitor_THT:C_Disc_D4.3mm_W1.9mm_P5.00mm"

Commit message: Mounting holes to schematic
Parts:
- added H1, H2, H3, H4: MountingHole, MountingHole:MountingHole_3.2mm_M3_Pad, symbol Mechanical:MountingHole

Commit message: Trace complete? Perhaps...
Parts:
- removed H1, H2, H3, H4: MountingHole, MountingHole:MountingHole_3.2mm_M3_Pad, symbol Mechanical:MountingHole
- added H1, H2, H3, H4: MountingHole_Pad, MountingHole:MountingHole_3.2mm_M3_Pad, symbol Mechanical:MountingHole_Pad
Connections:
- net GND: now also H1.1, H2.1, H3.1, H4.1
