File: led-output-board.kicad_pcb (KiCad board)
At the start: 2 copper layers, 80.9 x 96.4 mm, 29 parts, among them J1 DBT50G-9.5-2P, J10 DB301V-3.5-3P-GN, J2 Conn_02x08_Odd_Even, J3 DB301V-3.5-3P-GN, J4 DB301V-3.5-3P-GN, J5 DB301V-3.5-3P-GN, J6 DB301V-3.5-3P-GN, J7 DB301V-3.5-3P-GN, J8 DB301V-3.5-3P-GN, J9 DB301V-3.5-3P-GN, U1 SN74LVC8T245PWR

Commit message: Trace complete? Perhaps...
Parts:
- added H1: MountingHole_Pad, MountingHole:MountingHole_3.2mm_M3_Pad, F.Cu at (90.2, 70.4)
- added H2: MountingHole_Pad, MountingHole:MountingHole_3.2mm_M3_Pad, F.Cu at (110.5, 156.2)
- added H3: MountingHole_Pad, MountingHole:MountingHole_3.2mm_M3_Pad, F.Cu at (67.3, 70.3)
- added H4: MountingHole_Pad, MountingHole:MountingHole_3.2mm_M3_Pad, F.Cu at (67.3, 156.4)
- moved F3 0.25 mm to (127.3, 92.4)
- moved F8 0.25 mm to (127.2, 151.4)
- moved F7 0.25 mm to (127.3, 139.7)
- moved F5 0.23 mm to (127.1, 116.0)
- moved F6 0.23 mm to (127.2, 127.8)
- moved F2 0.17 mm to (127.3, 80.5)
- moved F4 0.14 mm to (127.2, 104.2)
Routing:
- net Net-(J10-Pad2): track 0.00 -> 51.2 mm, vias 0 -> 2
- net Net-(J9-Pad2): track 0.00 -> 48.7 mm, vias 0 -> 2
- net Net-(J3-Pad2): track 0.00 -> 44.9 mm, vias 0 -> 2
- net Net-(J4-Pad2): track 0.00 -> 42.6 mm, vias 0 -> 2
- net Net-(J8-Pad2): track 0.00 -> 41.6 mm, vias 0 -> 2
- net Net-(J5-Pad2): track 0.00 -> 40.1 mm, vias 0 -> 2
- net Net-(J7-Pad2): track 0.00 -> 38.5 mm, vias 0 -> 2
- net Net-(J6-Pad2): track 0.00 -> 37.8 mm, vias 0 -> 2
- net Net-(F5-Pad2): track 0.00 -> 8.02 mm
- net Net-(F6-Pad2): track 0.00 -> 8.02 mm
- net Net-(F4-Pad2): track 0.00 -> 8.01 mm
- net Net-(F8-Pad2): track 0.00 -> 7.95 mm
- net Net-(F1-Pad2): track 0.00 -> 7.94 mm
- net Net-(F3-Pad2): track 0.00 -> 7.91 mm
- net Net-(F7-Pad2): track 0.00 -> 7.90 mm
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
Commit message: Silkscreen additions
Parts:
- added G***: LOGO, Project Libraries:LEDGuy, F.Cu at (78.6, 142.3)
- J2: value Conn_02x08_Odd_Even -> Data Input
- U1: value SN74LVC8T245PWR -> Level Shifter
- moved H2 2.75 mm to (113.2, 156.2)
- moved J1 1.06 mm to (106.0, 72.4)
- moved F1 0.88 mm to (126.4, 69.0)
- moved F2 0.88 mm to (126.5, 80.8)
- moved F3 0.88 mm to (126.4, 92.6)
- moved F7 0.88 mm to (126.4, 139.9)
- moved F6 0.88 mm to (126.3, 128.0)
- moved F4 0.88 mm to (126.3, 104.4)
- moved F5 0.88 mm to (126.3, 116.3)
- moved F8 0.88 mm to (126.4, 151.7)
- moved J10 0.88 mm to (136.8, 155.2)
- moved J3 0.88 mm to (136.8, 72.5)
- moved J4 0.88 mm to (136.8, 84.3)
- moved J5 0.88 mm to (136.8, 96.2)
- moved J6 0.88 mm to (136.8, 108.0)
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Routing:
- net Net-(J6-Pad2): track 37.8 -> 36.8 mm
- net Net-(J3-Pad2): track 44.9 -> 44.0 mm
- net Net-(J5-Pad2): track 40.1 -> 39.3 mm
- net Net-(J7-Pad2): track 38.5 -> 37.8 mm
- net Net-(J10-Pad2): track 51.2 -> 50.5 mm
Other:
- board text added: "+"
- board text added: "-"
- board text added: "1"
- board text added: "100nF"
- board text added: "15"
- board text added: "16"
- board text added: "2"
- board text added: "D"
- board text added: "LED Output Board v1.0"

Commit message: DRC passes no errors or warnings
Routing:
- net Net-(J4-Pad2): track 42.6 -> 41.6 mm
Other:
- board text added: "47Ω"
- board text added: "Strip 1"
- board text added: "Strip 8"
Changed lines of the file:
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@@
 			(at 0 -4 0)
 			(layer "F.SilkS")
+			(hide yes)
 			(effects
 				(font
@@
 			(at 0 0 0)
 			(layer "F.SilkS")
+			(hide yes)
 			(effects
 				(font
@@
 		)
 	)
+	(gr_text "Strip 1"
+		(at 127.55 76.35 0)
+		(layer "F.SilkS")
+		(effects
+			(font
+				(size 1 1)
+				(thickness 0.2)
+				(bold yes)
+			)
+			(justify left bottom)
+		)
+	)
+	(gr_text "Strip 8"
+		(at 127.65 158.6 0)
+		(layer "F.SilkS")
+		(effects
+			(font
+				(size 1 1)
+				(thickness 0.2)
+				(bold yes)
+			)
+			(justify left bottom)
+		)
+	)
 	(gr_text "D"
 		(at 141.85 73.25 90)
@@
 		)
 	)
+	(gr_text "47Ω"
+		(at 97.3 89.65 0)
+		(layer "F.SilkS")
+		(effects
+			(font
+				(size 1.5 1.5)
+				(thickness 0.3)
+				(bold yes)
+			)
+			(justify left bottom)
+		)
+	)
 	(gr_text "-"
 		(at 99.75 67.8 0)
@@
 	)
 	(segment
-		(start 111.6 88.75)
-		(end 111.45 88.75)
+		(start 111.45 88.75)
+		(end 111.600001 88.75)
 		(width 0.2)
 		(layer "B.Cu")
@@
 	)
 	(segment
-		(start 116.25 84.1)
-		(end 111.6 88.75)
+		(start 111.600001 88.75)
+		(end 116.010358 84.339643)
 		(width 0.2)
 		(layer "B.Cu")
@@
 	)
 	(segment
-		(start 129.45 84.339643)
-		(end 115.4 84.339643)
+		(start 116.010358 84.339643)
+		(end 129.45 84.339643)
 		(width 0.2)
 		(layer "B.Cu")

Commit message: Maybe time to send it?
Parts:
- moved G*** 6.17 mm to (82.3, 147.2)
- moved H2 1.03 mm to (114.0, 156.9)
- moved H4 0.92 mm to (66.7, 156.9)
Other:
- board text added: "Data Input"
- board text added: "Level Shifter"
Changed lines of the file:
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@@
 			(at 1.2 27.18 0)
 			(layer "F.Fab")
+			(hide yes)
 			(effects
 				(font
@@
 	(footprint "MountingHole:MountingHole_3.2mm_M3_Pad"
 		(layer "F.Cu")
-		(at 113.2 156.25)
+		(at 113.95 156.95)
 		(descr "Mounting Hole 3.2mm, M3, generated by kicad-footprint-generator mountinghole.py")
 		(tags "mountinghole M3")
@@
 	(footprint "Project Libraries:LEDGuy"
 		(layer "F.Cu")
-		(at 78.6 142.3)
+		(at 82.35 147.2)
 		(property "Reference" "G***"
 			(at 0 0 0)
@@
 			(at 6.53 0.08 180)
 			(layer "F.Fab")
+			(hide yes)
 			(effects
 				(font
@@
 	(footprint "MountingHole:MountingHole_3.2mm_M3_Pad"
 		(layer "F.Cu")
-		(at 67.3 156.25)
+		(at 66.7 156.95)
 		(descr "Mounting Hole 3.2mm, M3, generated by kicad-footprint-generator mountinghole.py")
 		(tags "mountinghole M3")
@@
 		(layer "Edge.Cuts")
 	)
+	(gr_text "Data Input"
+		(at 64.1 131.1 0)
+		(layer "F.SilkS")
+		(effects
+			(font
+				(size 1 1)
+				(thickness 0.2)
+				(bold yes)
+			)
+			(justify left bottom)
+		)
+	)
+	(gr_text "Level Shifter"
+		(at 81.25 119.9 0)
+		(layer "F.SilkS")
+		(effects
+			(font
+				(size 1 1)
+				(thickness 0.2)
+				(bold yes)
+			)
+			(justify left bottom)
+		)
+	)
 	(gr_text "LED Output Board\nv1.0"
-		(at 87.1 144.15 0)
+		(at 90.85 149.05 0)
 		(layer "F.SilkS")
 		(effects
@@
 	)
 	(segment
-		(start 108.65 96.1)
-		(end 100.95 103.8)
+		(start 110.439643 96.15)
+		(end 108.6 96.15)
 		(width 0.2)
 		(layer "F.Cu")
@@
 	)
 	(segment
-		(start 110.45 96.139643)
-		(end 110.410357 96.1)
+		(start 108.6 96.15)
+		(end 100.95 103.8)
 		(width 0.2)
 		(layer "F.Cu")
@@
 	)
 	(segment
-		(start 129.45 96.139643)
-		(end 129.9 96.139643)
+		(start 110.45 96.139643)
+		(end 110.439643 96.15)
 		(width 0.2)
 		(layer "F.Cu")
@@
 	)
 	(segment
-		(start 129.917245 96.156888)
-		(end 136.85 96.156888)
+		(start 129.45 96.139643)
+		(end 129.9 96.139643)
 		(width 0.2)
 		(layer "F.Cu")
@@
 	)
 	(segment
-		(start 110.410357 96.1)
-		(end 108.65 96.1)
+		(start 129.917245 96.156888)
+		(end 136.85 96.156888)
 		(width 0.2)
 		(layer "F.Cu")
@@
 	)
 	(segment
-		(start 110.35 96.139643)
+		(start 110.45 96.139643)
 		(end 129.45 96.139643)
 		(width 0.2)
